File: TextTest.kicad_sch (KiCad schematic)
At the start: 0 parts

Commit message: updates
Other:
- note added: "01234567890123456789"
Changed lines of the file:
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@@
     (effects (font (size 1.27 1.27) (thickness 0.254) bold italic) (justify left bottom))
+  )
+  (text "01234567890123456789" (at 144.145 120.65 0)
+    (effects (font (size 1.27 1.27)) (justify right bottom))
   )
   (text "Text: Left Aligned - Italic - 1.27 - Vertical" (at 93.98 107.315 90)
@@
     (effects (font (size 1.27 1.27)) (justify right bottom))
   )
+  (text "01234567890123456789" (at 120.015 118.745 0)
+    (effects (font (size 1.27 1.27)) (justify left bottom))
+  )
   (text "Text: Left Aligned - Bold Italic - 1.27 - Horizontal"
