File: TextTest.kicad_sch (KiCad schematic)
At the start: 0 parts

Commit message: updates
Other:
- note added: "ABCDEFGHIJKLMNOPQRSTUVWXYZ 0123456789-_"
Changed lines of the file:
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@@
 (kicad_sch (version 20230121) (generator eeschema)
   (paper "A4")
-  (no_connect (at 262.89 48.895))
+  (no_connect (at 280.035 46.99))
   (no_connect (at 64.135 51.435))
-  (no_connect (at 264.795 125.095))
+  (no_connect (at 280.67 126.365))
   (no_connect (at 60.96 127.635))
   (polyline (pts (xy 120.65 69.85) (xy 120.65 106.68))
@@
     (effects (font (size 1.27 1.27)) (justify left top))
   )
+  (text "ABCDEFGHIJKLMNOPQRSTUVWXYZ 0123456789-_" (at 231.14 86.36 0)
+    (effects (font (size 1.27 1.27) bold) (justify right bottom))
+  )
   (text "Text: Left Aligned - Bold - 1.27 - Vertical" (at 83.185 107.315 90)
     (effects (font (size 1.27 1.27) (thickness 0.254) bold) (justify left bottom))
+  )
+  (text "ABCDEFGHIJKLMNOPQRSTUVWXYZ 0123456789-_" (at 230.505 106.68 0)
+    (effects (font (size 1.27 1.27) bold italic) (justify right bottom))
+  )
+  (text "ABCDEFGHIJKLMNOPQRSTUVWXYZ 0123456789-_" (at 184.785 101.6 0)
+    (effects (font (size 1.27 1.27) (thickness 0.254) bold italic) (justify left bottom))
+  )
+  (text "ABCDEFGHIJKLMNOPQRSTUVWXYZ 0123456789-_" (at 271.145 107.315 90)
+    (effects (font (size 1.27 1.27) (thickness 0.254) bold italic) (justify left bottom))
+  )
+  (text "ABCDEFGHIJKLMNOPQRSTUVWXYZ 0123456789-_" (at 184.785 71.12 0)
+    (effects (font (size 1.27 1.27)) (justify left bottom))
   )
   (text "Text: Right Aligned - Bold - 1.27 - Vertical" (at 88.9 62.865 90)
@@
     (effects (font (size 1.27 1.27)) (justify left bottom))
   )
+  (text "ABCDEFGHIJKLMNOPQRSTUVWXYZ 0123456789-_" (at 184.785 81.28 0)
+    (effects (font (size 1.27 1.27) (thickness 0.254) bold) (justify left bottom))
+  )
+  (text "ABCDEFGHIJKLMNOPQRSTUVWXYZ 0123456789-_" (at 249.555 107.315 90)
+    (effects (font (size 1.27 1.27) (thickness 0.254) bold) (justify left bottom))
+  )
+  (text "ABCDEFGHIJKLMNOPQRSTUVWXYZ 0123456789-_" (at 266.065 61.595 90)
+    (effects (font (size 1.27 1.27) italic) (justify right bottom))
+  )
   (text "Text: Left Aligned - Normal - 1.27 - Horizontal" (at 120.65 71.12 0)
+    (effects (font (size 1.27 1.27)) (justify left bottom))
+  )
+  (text "ABCDEFGHIJKLMNOPQRSTUVWXYZ 0123456789-_" (at 184.785 91.44 0)
+    (effects (font (size 1.27 1.27) italic) (justify left bottom))
+  )
+  (text "ABCDEFGHIJKLMNOPQRSTUVWXYZ 0123456789-_" (at 239.395 107.315 90)
     (effects (font (size 1.27 1.27)) (justify left bottom))
   )
@@
     (at 104.775 107.315 90)
     (effects (font (size 1.27 1.27) (thickness 0.254) bold italic) (justify left bottom))
+  )
+  (text "ABCDEFGHIJKLMNOPQRSTUVWXYZ 0123456789-_" (at 230.505 96.52 0)
+    (effects (font (size 1.27 1.27) italic) (justify right bottom))
   )
   (text "01234567890123456789" (at 144.145 120.65 0)
@@
     (effects (font (size 1.27 1.27)) (justify right bottom))
   )
+  (text "ABCDEFGHIJKLMNOPQRSTUVWXYZ 0123456789-_" (at 231.14 76.2 0)
+    (effects (font (size 1.27 1.27)) (justify right bottom))
+  )
   (text "Text: Right Aligned - Italic - 1.27 - Vertical" (at 99.695 62.865 90)
     (effects (font (size 1.27 1.27) italic) (justify right bottom))
@@
   (text "Text: Right Aligned - Normal - 1.27 - Horizontal" (at 78.105 57.785 90)
     (effects (font (size 1.27 1.27)) (justify right bottom))
+  )
+  (text "ABCDEFGHIJKLMNOPQRSTUVWXYZ 0123456789-_" (at 244.475 60.96 90)
+    (effects (font (size 1.27 1.27)) (justify right bottom))
+  )
+  (text "ABCDEFGHIJKLMNOPQRSTUVWXYZ 0123456789-_" (at 260.35 107.315 90)
+    (effects (font (size 1.27 1.27) italic) (justify left bottom))
   )
   (text "01234567890123456789" (at 120.015 118.745 0)
@@
     (at 120.65 101.6 0)
     (effects (font (size 1.27 1.27) (thickness 0.254) bold italic) (justify left bottom))
+  )
+  (text "ABCDEFGHIJKLMNOPQRSTUVWXYZ 0123456789-_" (at 276.86 61.595 90)
+    (effects (font (size 1.27 1.27) bold italic) (justify right bottom))
   )
   (text "Text: Right Aligned - Bold - 1.27 - Horizontal" (at 167.64 86.36 0)
@@
     (effects (font (size 1.27 1.27) bold italic) (justify right bottom))
   )
+  (text "ABCDEFGHIJKLMNOPQRSTUVWXYZ 0123456789-_" (at 255.27 60.96 90)
+    (effects (font (size 1.27 1.27) bold) (justify right bottom))
+  )
   (sheet_instances
