File: TextTest.kicad_sch (KiCad schematic)
At the start: 0 parts

Commit message: updates
Other:
- note added: "A B C D E F G H I J K L M 0 1 2 3 4 5"
Changed lines of the file:
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@@
 (kicad_sch (version 20230121) (generator eeschema)
   (paper "A4")
-  (no_connect (at 280.035 46.99))
-  (no_connect (at 64.135 51.435))
-  (no_connect (at 280.67 126.365))
+  (no_connect (at 282.575 13.335))
+  (no_connect (at 64.77 13.335))
+  (no_connect (at 282.575 126.365))
   (no_connect (at 60.96 127.635))
   (polyline (pts (xy 120.65 69.85) (xy 120.65 106.68))
@@
     (effects (font (size 1.27 1.27) (thickness 0.254) bold italic) (justify left bottom))
   )
+  (text "A B C D E F G H I J K L M 0 1 2 3 4 5" (at 225.425 47.625 0)
+    (effects (font (size 1.27 1.27) italic) (justify right bottom))
+  )
   (text "ABCDEFGHIJKLMNOPQRSTUVWXYZ 0123456789-_" (at 271.145 107.315 90)
     (effects (font (size 1.27 1.27) (thickness 0.254) bold italic) (justify left bottom))
   )
+  (text "A B C D E F G H I J K L M 0 1 2 3 4 5" (at 239.395 57.15 90)
+    (effects (font (size 1.27 1.27)) (justify left bottom))
+  )
   (text "ABCDEFGHIJKLMNOPQRSTUVWXYZ 0123456789-_" (at 184.785 71.12 0)
+    (effects (font (size 1.27 1.27)) (justify left bottom))
+  )
+  (text "A B C D E F G H I J K L M 0 1 2 3 4 5" (at 186.055 22.225 0)
     (effects (font (size 1.27 1.27)) (justify left bottom))
   )
@@
   )
   (text "Text: Right Aligned - Italic - 1.27 - Horizontal" (at 167.64 96.52 0)
+    (effects (font (size 1.27 1.27) italic) (justify right bottom))
+  )
+  (text "A B C D E F G H I J K L M 0 1 2 3 4 5" (at 255.905 17.78 90)
+    (effects (font (size 1.27 1.27) bold) (justify right bottom))
+  )
+  (text "A B C D E F G H I J K L M 0 1 2 3 4 5" (at 244.475 17.78 90)
+    (effects (font (size 1.27 1.27)) (justify right bottom))
+  )
+  (text "A B C D E F G H I J K L M 0 1 2 3 4 5" (at 186.055 42.545 0)
+    (effects (font (size 1.27 1.27) italic) (justify left bottom))
+  )
+  (text "A B C D E F G H I J K L M 0 1 2 3 4 5" (at 265.43 17.78 90)
     (effects (font (size 1.27 1.27) italic) (justify right bottom))
   )
@@
     (effects (font (size 1.27 1.27) italic) (justify right bottom))
   )
+  (text "A B C D E F G H I J K L M 0 1 2 3 4 5" (at 249.555 57.15 90)
+    (effects (font (size 1.27 1.27) (thickness 0.254) bold) (justify left bottom))
+  )
   (text "Text: Left Aligned - Normal - 1.27 - Horizontal" (at 120.65 71.12 0)
     (effects (font (size 1.27 1.27)) (justify left bottom))
@@
     (effects (font (size 1.27 1.27) italic) (justify left bottom))
   )
+  (text "A B C D E F G H I J K L M 0 1 2 3 4 5" (at 276.86 17.78 90)
+    (effects (font (size 1.27 1.27) bold italic) (justify right bottom))
+  )
   (text "ABCDEFGHIJKLMNOPQRSTUVWXYZ 0123456789-_" (at 239.395 107.315 90)
     (effects (font (size 1.27 1.27)) (justify left bottom))
+  )
+  (text "A B C D E F G H I J K L M 0 1 2 3 4 5" (at 186.055 52.705 0)
+    (effects (font (size 1.27 1.27) (thickness 0.254) bold italic) (justify left bottom))
   )
   (text "Text: Left Aligned - Italic - 1.27 - Horizontal" (at 120.65 91.44 0)
@@
     (at 104.775 107.315 90)
     (effects (font (size 1.27 1.27) (thickness 0.254) bold italic) (justify left bottom))
+  )
+  (text "A B C D E F G H I J K L M 0 1 2 3 4 5" (at 225.425 37.465 0)
+    (effects (font (size 1.27 1.27) bold) (justify right bottom))
   )
   (text "ABCDEFGHIJKLMNOPQRSTUVWXYZ 0123456789-_" (at 230.505 96.52 0)
@@
     (effects (font (size 1.27 1.27)) (justify right bottom))
   )
+  (text "A B C D E F G H I J K L M 0 1 2 3 4 5" (at 271.145 57.15 90)
+    (effects (font (size 1.27 1.27) (thickness 0.254) bold italic) (justify left bottom))
+  )
+  (text "A B C D E F G H I J K L M 0 1 2 3 4 5" (at 186.055 32.385 0)
+    (effects (font (size 1.27 1.27) (thickness 0.254) bold) (justify left bottom))
+  )
   (text "Text: Right Aligned - Italic - 1.27 - Vertical" (at 99.695 62.865 90)
     (effects (font (size 1.27 1.27) italic) (justify right bottom))
@@
   )
   (text "ABCDEFGHIJKLMNOPQRSTUVWXYZ 0123456789-_" (at 244.475 60.96 90)
+    (effects (font (size 1.27 1.27)) (justify right bottom))
+  )
+  (text "A B C D E F G H I J K L M 0 1 2 3 4 5" (at 225.425 27.305 0)
     (effects (font (size 1.27 1.27)) (justify right bottom))
   )
@@
     (effects (font (size 1.27 1.27) (thickness 0.254) bold) (justify left bottom))
   )
+  (text "A B C D E F G H I J K L M 0 1 2 3 4 5" (at 225.425 57.785 0)
+    (effects (font (size 1.27 1.27) bold italic) (justify right bottom))
+  )
+  (text "A B C D E F G H I J K L M 0 1 2 3 4 5" (at 260.35 57.15 90)
+    (effects (font (size 1.27 1.27) italic) (justify left bottom))
+  )
   (text "Text: Right Aligned - Bold Italic - 1.27 - Vertical"
